Commit message: Add controllers for freight robot and a teleop launch

File: robots/freight.gazebo.xacro (robot description, xacro)
@@ -1,3 +1,63 @@
 <robot xmlns:xacro="http://www.ros.org/wiki/xacro" name="freight" >
   <xacro:include filename="$(find fetch_description)/robots/freight.urdf" />
+  <!-- Base is modeled as a big tub sitting on floor, with two wheels -->
+<!--   <gazebo reference="base_link">
+    <kp>100000000.0</kp>
+    <kd>10.0</kd>
+    <mu1>0.1</mu1>
+    <mu2>0.1</mu2>
+    <fdir1>1 0 0</fdir1>
+    <maxVel>10.0</maxVel>
+    <minDepth>0.0005</minDepth>
+  </gazebo>
+  <gazebo reference="r_wheel_link">
+    <kp>500000.0</kp>
+    <kd>10.0</kd>
+    <mu1>10</mu1>
+    <mu2>10</mu2>
+    <fdir1>1 0 0</fdir1>
+    <maxVel>1.0</maxVel>
+    <minDepth>0.003</minDepth>
+    <material>Gazebo/Black</material>
+  </gazebo>
+  <gazebo reference="l_wheel_link">
+    <kp>500000.0</kp>
+    <kd>10.0</kd>
+    <mu1>10</mu1>
+    <mu2>10</mu2>
+    <fdir1>1 0 0</fdir1>
+    <maxVel>1.0</maxVel>
+    <minDepth>0.003</minDepth>
+    <material>Gazebo/Black</material>
+  </gazebo>
+  <gazebo reference="l_wheel_joint">
+    <implicitSpringDamper>1</implicitSpringDamper>
+  </gazebo>
+  <gazebo reference="r_wheel_joint">
+    <implicitSpringDamper>1</implicitSpringDamper>
+  </gazebo> -->
+  <!-- adding transmissions for the wheel joint to apply default ros_control plugin -->
+  <transmission name="l_wheel_trans">
+  	<type>transmission_interface/SimpleTransmission</type>
+  	<joint name="l_wheel_joint">
+      <hardwareInterface>VelocityJointInterface</hardwareInterface>
+  	</joint>
+  	<actuator name="l_wheel_motor">
+      <mechanicalReduction>1</mechanicalReduction>
+  	</actuator>
+  </transmission>
+  <transmission name="r_wheel_trans">
+  	<type>transmission_interface/SimpleTransmission</type>
+  	<joint name="r_wheel_joint">
+      <hardwareInterface>VelocityJointInterface</hardwareInterface>
+  	</joint>
+  	<actuator name="r_wheel_motor">
+      <mechanicalReduction>1</mechanicalReduction>
+  	</actuator>
+  </transmission>
+  <!-- Gazebo plugin for ROS Control -->
+  <gazebo>
+    <plugin name="gazebo_ros_control" filename="libgazebo_ros_control.so">
+    </plugin>
+  </gazebo>
 </robot>
