Commit message: Add fetch robot configuration. Now the application can spawn multiple fetch robots and controll the whells and joints

File: robots/fetch.gazebo.xacro (robot description, xacro)
@@ -105,3 +105,170 @@
     <material>Gazebo/Grey</material>
   </gazebo>
+  <!-- adding transmissions for the wheel joints and other joints to apply default ros_control plugin -->
+  <transmission name="l_wheel_trans">
+  	<type>transmission_interface/SimpleTransmission</type>
+  	<joint name="l_wheel_joint">
+      <hardwareInterface>hardware_interface/VelocityJointInterface</hardwareInterface>
+  	</joint>
+  	<actuator name="l_wheel_motor">
+      <mechanicalReduction>1</mechanicalReduction>
+  	</actuator>
+  </transmission>
+  <transmission name="r_wheel_trans">
+  	<type>transmission_interface/SimpleTransmission</type>
+  	<joint name="r_wheel_joint">
+      <hardwareInterface>hardware_interface/VelocityJointInterface</hardwareInterface>
+  	</joint>
+  	<actuator name="r_wheel_motor">
+      <mechanicalReduction>1</mechanicalReduction>
+  	</actuator>
+  </transmission>
+  <transmission name="torso_lift_trans">
+  	<type>transmission_interface/SimpleTransmission</type>
+  	<joint name="torso_lift_joint">
+      <hardwareInterface>hardware_interface/PositionJointInterface</hardwareInterface>
+  	</joint>
+  	<actuator name="torso_lift_motor">
+      <mechanicalReduction>1</mechanicalReduction>
+  	</actuator>
+  </transmission>
+  <transmission name="head_pan_trans">
+    <type>transmission_interface/SimpleTransmission</type>
+    <joint name="head_pan_joint">
+      <hardwareInterface>hardware_interface/EffortJointInterface</hardwareInterface>
+    </joint>
+    <actuator name="head_pan_motor">
+      <hardwareInterface>EffortJointInterface</hardwareInterface>
+      <mechanicalReduction>1</mechanicalReduction>
+    </actuator>
+  </transmission>
+  <transmission name="head_tilt_trans">
+    <type>transmission_interface/SimpleTransmission</type>
+    <joint name="head_tilt_joint">
+      <hardwareInterface>hardware_interface/EffortJointInterface</hardwareInterface>
+    </joint>
+    <actuator name="head_tilt_motor">
+      <hardwareInterface>EffortJointInterface</hardwareInterface>
+      <mechanicalReduction>1</mechanicalReduction>
+    </actuator>
+  </transmission>
+  <transmission name="shoulder_pan_trans">
+    <type>transmission_interface/SimpleTransmission</type>
+    <joint name="shoulder_pan_joint">
+      <hardwareInterface>hardware_interface/EffortJointInterface</hardwareInterface>
+    </joint>
+    <actuator name="shoulder_pan_motor">
+      <hardwareInterface>EffortJointInterface</hardwareInterface>
+      <mechanicalReduction>1</mechanicalReduction>
+    </actuator>
+  </transmission>
+  <transmission name="shoulder_lift_trans">
+    <type>transmission_interface/SimpleTransmission</type>
+    <joint name="shoulder_lift_joint">
+      <hardwareInterface>hardware_interface/EffortJointInterface</hardwareInterface>
+    </joint>
+    <actuator name="shoulder_lift_motor">
+      <hardwareInterface>EffortJointInterface</hardwareInterface>
+      <mechanicalReduction>1</mechanicalReduction>
+    </actuator>
+  </transmission>
+  <transmission name="upperarm_roll_trans">
+    <type>transmission_interface/SimpleTransmission</type>
+    <joint name="upperarm_roll_joint">
+      <hardwareInterface>hardware_interface/EffortJointInterface</hardwareInterface>
+    </joint>
+    <actuator name="upperarm_roll_motor">
+      <hardwareInterface>EffortJointInterface</hardwareInterface>
+      <mechanicalReduction>1</mechanicalReduction>
+    </actuator>
+  </transmission>
+  <transmission name="elbow_flex_trans">
+    <type>transmission_interface/SimpleTransmission</type>
+    <joint name="elbow_flex_joint">
+      <hardwareInterface>hardware_interface/EffortJointInterface</hardwareInterface>
+    </joint>
+    <actuator name="elbow_flex_motor">
+      <hardwareInterface>EffortJointInterface</hardwareInterface>
+      <mechanicalReduction>1</mechanicalReduction>
+    </actuator>
+  </transmission>
+  <transmission name="forearm_roll_trans">
+    <type>transmission_interface/SimpleTransmission</type>
+    <joint name="forearm_roll_joint">
+      <hardwareInterface>hardware_interface/EffortJointInterface</hardwareInterface>
+    </joint>
+    <actuator name="forearm_roll_motor">
+      <hardwareInterface>EffortJointInterface</hardwareInterface>
+      <mechanicalReduction>1</mechanicalReduction>
+    </actuator>
+  </transmission>
+  <transmission name="wrist_flex_trans">
+    <type>transmission_interface/SimpleTransmission</type>
+    <joint name="wrist_flex_joint">
+      <hardwareInterface>hardware_interface/EffortJointInterface</hardwareInterface>
+    </joint>
+    <actuator name="wrist_flex_motor">
+      <hardwareInterface>EffortJointInterface</hardwareInterface>
+      <mechanicalReduction>1</mechanicalReduction>
+    </actuator>
+  </transmission>
+  <transmission name="wrist_roll_trans">
+    <type>transmission_interface/SimpleTransmission</type>
+    <joint name="wrist_roll_joint">
+      <hardwareInterface>hardware_interface/EffortJointInterface</hardwareInterface>
+    </joint>
+    <actuator name="wrist_roll_motor">
+      <hardwareInterface>EffortJointInterface</hardwareInterface>
+      <mechanicalReduction>1</mechanicalReduction>
+    </actuator>
+  </transmission>
+  <!-- SICK TIM561 (25m Range) -->
+  <gazebo reference="laser_link">
+    <sensor type="ray" name="base_laser">
+      <pose>0 0 0 0 0 0</pose>
+      <visualize>false</visualize>
+      <update_rate>15</update_rate>
+      <ray>
+        <scan>
+          <horizontal>
+            <samples>662</samples>
+            <resolution>1</resolution>
+            <min_angle>-1.91986</min_angle>
+            <max_angle>1.91986</max_angle>
+          </horizontal>
+        </scan>
+        <range>
+          <min>0.05</min>
+          <max>25.0</max>
+          <resolution>0.01</resolution>
+        </range>
+        <noise>
+          <!-- Noise parameters based on spec for SICK TIM561 (10m version) -->
+          <type>gaussian</type>
+          <mean>0.0</mean>
+          <stddev>0.02</stddev>
+        </noise>
+      </ray>
+      <plugin name="gazebo_ros_base_hokuyo_controller" filename="libgazebo_ros_laser.so">
+        <topicName>/base_scan</topicName>
+        <frameName>laser_link</frameName>
+      </plugin>
+    </sensor>
+  </gazebo>
+  <!-- Color the bellows -->
+  <gazebo reference="bellows_link">
+    <material>Gazebo/Black</material>
+  </gazebo>
+  <gazebo reference="bellows_link2">
+    <material>Gazebo/Black</material>
+  </gazebo>
+  <!-- Color the estop -->
+  <gazebo reference="estop_link">
+    <material>Gazebo/Red</material>
+  </gazebo>
+  <!-- Load the plugin -->
+  <gazebo>
+    <plugin name="gazebo_ros_control" filename="libgazebo_ros_control.so">
+    </plugin>
+  </gazebo>
 </robot>

File: robots/freight.gazebo.xacro (robot description, xacro)
@@ -45,5 +45,5 @@
   	<type>transmission_interface/SimpleTransmission</type>
   	<joint name="l_wheel_joint">
-      <hardwareInterface>VelocityJointInterface</hardwareInterface>
+      <hardwareInterface>hardware_interface/VelocityJointInterface</hardwareInterface>
   	</joint>
   	<actuator name="l_wheel_motor">
@@ -54,5 +54,5 @@
   	<type>transmission_interface/SimpleTransmission</type>
   	<joint name="r_wheel_joint">
-      <hardwareInterface>VelocityJointInterface</hardwareInterface>
+      <hardwareInterface>hardware_interface/VelocityJointInterface</hardwareInterface>
   	</joint>
   	<actuator name="r_wheel_motor">
@@ -64,5 +64,5 @@
     <sensor type="ray" name="base_laser">
       <pose>0 0 0 0 0 0</pose>
-      <visualize>true</visualize>
+      <visualize>false</visualize>
       <update_rate>15</update_rate>
       <ray>
@@ -93,4 +93,8 @@
     </sensor>
   </gazebo>
+  <!-- Color the estop -->
+  <gazebo reference="estop_link">
+    <material>Gazebo/Red</material>
+  </gazebo>
   <!-- Gazebo plugin for ROS Control -->
   <gazebo>

Commit message: add fetch arm initialization feature. Add navigation feature for fetch. Now we can respawn multiple fetch and freight robots

File: robots/fetch.gazebo.xacro (robot description, xacro)
@@ -105,4 +105,29 @@
     <material>Gazebo/Grey</material>
   </gazebo>
+  <!-- turn off the gravity for arm links -->
+  <gazebo reference="shoulder_pan_link">
+    <gravity>0</gravity>
+  </gazebo>
+  <gazebo reference="shoulder_lift_link">
+    <gravity>0</gravity>
+  </gazebo>
+  <gazebo reference="upperarm_roll_link">
+    <gravity>0</gravity>
+  </gazebo>
+  <gazebo reference="elbow_flex_link">
+    <gravity>0</gravity>
+  </gazebo>
+  <gazebo reference="forearm_roll_link">
+    <gravity>0</gravity>
+  </gazebo>
+  <gazebo reference="wrist_flex_link">
+    <gravity>0</gravity>
+  </gazebo>
+  <gazebo reference="wrist_roll_link">
+    <gravity>0</gravity>
+  </gazebo>
+  <gazebo reference="gripper_link">
+    <gravity>0</gravity>
+  </gazebo>
   <!-- adding transmissions for the wheel joints and other joints to apply default ros_control plugin -->
   <transmission name="l_wheel_trans">
@@ -127,8 +152,8 @@
   	<type>transmission_interface/SimpleTransmission</type>
   	<joint name="torso_lift_joint">
-      <hardwareInterface>hardware_interface/PositionJointInterface</hardwareInterface>
+      <hardwareInterface>hardware_interface/EffortJointInterface</hardwareInterface>
   	</joint>
   	<actuator name="torso_lift_motor">
-      <hardwareInterface>PositionJointInterface</hardwareInterface>
+      <hardwareInterface>VelocityJointInterface</hardwareInterface>
       <mechanicalReduction>1</mechanicalReduction>
   	</actuator>
@@ -220,4 +245,34 @@
     </joint>
     <actuator name="wrist_roll_motor">
+      <hardwareInterface>EffortJointInterface</hardwareInterface>
+      <mechanicalReduction>1</mechanicalReduction>
+    </actuator>
+  </transmission>
+  <transmission name="r_gripper_finger_trans">
+    <type>transmission_interface/SimpleTransmission</type>
+    <joint name="r_gripper_finger_joint">
+      <hardwareInterface>hardware_interface/EffortJointInterface</hardwareInterface>
+    </joint>
+    <actuator name="r_gripper_finger_motor">
+      <hardwareInterface>EffortJointInterface</hardwareInterface>
+      <mechanicalReduction>1</mechanicalReduction>
+    </actuator>
+  </transmission>
+  <transmission name="l_gripper_finger_trans">
+    <type>transmission_interface/SimpleTransmission</type>
+    <joint name="l_gripper_finger_joint">
+      <hardwareInterface>hardware_interface/EffortJointInterface</hardwareInterface>
+    </joint>
+    <actuator name="l_gripper_finger_motor">
+      <hardwareInterface>EffortJointInterface</hardwareInterface>
+      <mechanicalReduction>1</mechanicalReduction>
+    </actuator>
+  </transmission>
+  <transmission name="bellows_trans">
+    <type>transmission_interface/SimpleTransmission</type>
+    <joint name="bellows_joint">
+      <hardwareInterface>hardware_interface/EffortJointInterface</hardwareInterface>
+    </joint>
+    <actuator name="bellows_motor">
       <hardwareInterface>EffortJointInterface</hardwareInterface>
       <mechanicalReduction>1</mechanicalReduction>
@@ -252,5 +307,5 @@
       </ray>
       <plugin name="gazebo_ros_base_hokuyo_controller" filename="libgazebo_ros_laser.so">
-        <topicName>/base_scan</topicName>
+        <topicName>base_scan</topicName>
         <frameName>laser_link</frameName>
       </plugin>

Commit message: rack tag models are now placed correctly. Now we can change robot base_link color

File: robots/fetch.gazebo.xacro (robot description, xacro)
@@ -1,4 +1,6 @@
 <robot xmlns:xacro="http://www.ros.org/wiki/xacro" name="fetch" >
   <xacro:include filename="$(find fetch_description)/robots/fetch.urdf" />
+  <xacro:arg name="color" default="Gray"/>
+  <xacro:property name="basecolor" value="$(arg color)" />
   <!-- Add four casters to the base -->
   <xacro:macro name="caster" params="prefix joint_x joint_y">
@@ -333,4 +335,8 @@
     <material>Gazebo/Red</material>
   </gazebo>
+  <!-- Color the base link -->
+  <gazebo reference="base_link">
+    <material>Gazebo/${basecolor}</material>
+  </gazebo>
   <!-- Load the plugin -->
   <gazebo>

File: robots/freight.gazebo.xacro (robot description, xacro)
@@ -1,4 +1,6 @@
 <robot xmlns:xacro="http://www.ros.org/wiki/xacro" name="freight" >
   <xacro:include filename="$(find fetch_description)/robots/freight.urdf" />
+  <xacro:arg name="color" default="Gray"/>
+  <xacro:property name="basecolor" value="$(arg color)" />
   <!-- Base is modeled as a big tub sitting on floor, with two wheels -->
   <gazebo reference="base_link">
@@ -97,4 +99,8 @@
     <material>Gazebo/Red</material>
   </gazebo>
+  <!-- Color the base link -->
+  <gazebo reference="base_link">
+    <material>Gazebo/${basecolor}</material>
+  </gazebo>
   <!-- Gazebo plugin for ROS Control -->
   <gazebo>
